Commit message: Separated serial from encoder code. Added a central Serial comms handler.

File: atlas_ws/src/atlas_python/resource/description/ros2_control.xacro (robot description, xacro)
@@ -1,7 +1,29 @@
 <xml version = "1.0"?>
 <robot xmlns:xacro="http://www.ros.org/wiki/xacro">
-    <ros2_control name = "atlasSystem" type = "system">
+    <!-- <ros2_control name = "atlasSystem" type = "system">
         <hardware>
             <plugin></plugin>
+            <param name =" "></param>
+        </hardware>
+        <joint name = "base_Lwheel_joint">
+            <command_interface name = "velocity">
+                <param name="min">-10</param>
+                <param name="max">10</param>
+            </command_interface>
+            <state_interfaace name = "velocity"/>
+            <state_interfaace name = "position"/>
+        </joint>
+        <joint name = "base_Rwheel_joint">
+            <command_interface name = "velocity">
+                <param name="min">-10</param>
+                <param name="max">10</param>
+            </command_interface>
+            <state_interfaace name = "velocity"/>
+            <state_interfaace name = "position"/>
+        </joint>
+    </ros2_control> -->
+    <ros2_control name = "GazeboSystem" type = "system">
+        <hardware>
+            <plugin>gazebo_ros2_control/GazeboSystem</plugin>
         </hardware>
         <joint name = "base_Lwheel_joint">
@@ -22,3 +44,9 @@
         </joint>
     </ros2_control>
+    <gazebo>
+        <plugin name = "gazebo_ros2_control" filename ="libgazebo_ros2_control.so">
+            <parameters>$(find atlas_python)/atlas_python/resource/config/my_controllers.yaml</parameters>
+            <!-- NOT SURE IF CORRECT PATH-->
+        </plugin>
+    </gazebo>
 </robot>
